Commit message: Update wheelchair.xacro

File: Graduation/wheelchair_gp_description/urdf/wheelchair.xacro (robot description, xacro)
@@ -380,5 +380,5 @@
       <origin xyz="0 0 0" rpy="0 0 0" />
       <geometry>
-        <mesh filename="package://wheelchair_gp_description2/meshes/laser_link.STL" />
+        <mesh filename="package://wheelchair_gp_description/meshes/laser_link.STL" />
       </geometry>
       <material name="">
@@ -389,5 +389,5 @@
       <origin xyz="0 0 0" rpy="0 0 0" />
       <geometry>
-        <mesh filename="package://wheelchair_gp_description2/meshes/laser_link.STL" />
+        <mesh filename="package://wheelchair_gp_description/meshes/laser_link.STL" />
       </geometry>
     </collision>
